Commit message: Initial version of R2 URDF.  Joints are in the right spot.  No decorations or colours added yet

File: r2_description/urdf/r2.urdf.xacro (robot description, xacro)
@@ -1,3 +1,84 @@
 <?xml version="1.0"?>
 <robot name="r2" xmlns:xacro="http://ros.org/wiki/xacro">
+  <link name="base_link">
+    <visual>
+      <origin xyz="0 0 0" rpy="0 0 0" />
+        <geometry>
+        <mesh filename="package://r2_description/meshes/R2_Feet.stl" scale="0.001 0.001 0.001"/>
+      </geometry>
+    </visual>
+  </link>
+  <joint name="ankle_joint" type="revolute">
+    <origin xyz="0 0 0.136726" rpy="0 0 0" />
+    <parent link="base_link" />
+    <child link="legs_link" />
+    <axis xyz="0 1 0" rpy="0 0 0" />
+    <limit effort="0" lower="0" upper="0.3054326" velocity="10.0" />
+  </joint>
+  <link name="legs_link">
+    <visual>
+      <origin xyz="0 0 -0.136726" rpy="0 0 0" />
+      <geometry>
+        <mesh filename="package://r2_description/meshes/R2_Legs.stl" scale="0.001 0.001 0.001"/>
+      </geometry>
+    </visual>
+  </link>
+  <joint name="shoulder_joint" type="revolute">
+    <origin xyz="0 0 0.56548" rpy="0 0 0" />
+    <parent link="legs_link" />
+    <child link="body_link" />
+    <axis xyz="0 1 0" rpy="0 0 0" />
+    <limit effort="0" lower="-0.6108652" upper="0" velocity="10.0" />
+  </joint>
+  <link name="body_link">
+    <visual>
+      <origin xyz="0 0 -0.702206" rpy="0 0 0" />
+      <geometry>
+        <mesh filename="package://r2_description/meshes/R2_Body.stl" scale="0.001 0.001 0.001"/>
+      </geometry>
+    </visual>
+  </link>
+  <joint name="neck_joint" type="revolute">
+    <origin xyz="0 0 0.12687" rpy="0 0 0" />
+    <parent link="body_link" />
+    <child link="dome_link" />
+    <axis xyz="0 0 1" rpy="0 0 0" />
+    <limit effort="0" lower="-3.14159" upper="3.14159" velocity="10.0" />
+  </joint>
+  <link name="dome_link">
+    <visual>
+      <origin xyz="0 0 -0.829076" rpy="0 0 0" />
+      <geometry>
+        <mesh filename="package://r2_description/meshes/R2_Dome.stl" scale="0.001 0.001 0.001"/>
+      </geometry>
+    </visual>
+  </link>
+  <joint name="center_leg_joint" type="fixed">
+    <origin xyz="0 0 -0.56548" rpy="0 0 0" />
+    <parent link="body_link" />
+    <child link="center_leg_link" />
+  </joint>
+  <link name="center_leg_link">
+    <visual>
+    <origin xyz="0 0 -0.136726" rpy="0 0 0" />
+      <geometry>
+        <mesh filename="package://r2_description/meshes/R2_CenterAnkle.stl" scale="0.001 0.001 0.001"/>
+      </geometry>
+    </visual>
+  </link>
+  <joint name="center_ankle_joint" type="revolute">
+    <origin xyz="0 0 0" rpy="0 0 0" />
+    <parent link="center_leg_link" />
+    <child link="center_foot_link" />
+    <axis xyz="0 1 0" rpy="0 0 0" />
+    <limit effort="0" lower="0" upper="0.3054326" velocity="10.0" />
+  </joint>
+  <link name="center_foot_link">
+    <visual>
+    <origin xyz="0 0 -0.136726" rpy="0 0 0" />
+      <geometry>
+        <mesh filename="package://r2_description/meshes/R2_Center_Foot.stl" scale="0.001 0.001 0.001"/>
+      </geometry>
+    </visual>
+  </link>
 </robot>

Commit message: Minor fixes for urdf

File: r2_description/urdf/r2.urdf.xacro (robot description, xacro)
@@ -7,4 +7,5 @@
         <mesh filename="package://r2_description/meshes/R2_Feet.stl" scale="0.001 0.001 0.001"/>
       </geometry>
+      <material name="Wite"> <color rgba="0.9 0.9 0.9 1.0"/> </material>
     </visual>
   </link>
@@ -22,4 +23,5 @@
         <mesh filename="package://r2_description/meshes/R2_Legs.stl" scale="0.001 0.001 0.001"/>
       </geometry>
+      <material name="Wite"> <color rgba="0.9 0.9 0.9 1.0"/> </material>
     </visual>
   </link>
@@ -37,4 +39,5 @@
         <mesh filename="package://r2_description/meshes/R2_Body.stl" scale="0.001 0.001 0.001"/>
       </geometry>
+      <material name="Wite"> <color rgba="0.9 0.9 0.9 1.0"/> </material>
     </visual>
   </link>
@@ -52,4 +55,5 @@
         <mesh filename="package://r2_description/meshes/R2_Dome.stl" scale="0.001 0.001 0.001"/>
       </geometry>
+      <material name="Wite"> <color rgba="0.9 0.9 0.9 1.0"/> </material>
     </visual>
   </link>
@@ -65,4 +69,5 @@
         <mesh filename="package://r2_description/meshes/R2_CenterAnkle.stl" scale="0.001 0.001 0.001"/>
       </geometry>
+      <material name="Wite"> <color rgba="0.9 0.9 0.9 1.0"/> </material>
     </visual>
   </link>
@@ -80,4 +85,5 @@
         <mesh filename="package://r2_description/meshes/R2_Center_Foot.stl" scale="0.001 0.001 0.001"/>
       </geometry>
+      <material name="Wite"> <color rgba="0.9 0.9 0.9 1.0"/> </material>
     </visual>
   </link>

Commit message: So many changes, none of which are tested: - added bringup - added control - added hardware interface for odrives - removed piper

File: r2_description/urdf/r2.urdf.xacro (robot description, xacro)
@@ -10,4 +10,20 @@
     </visual>
   </link>
+  <joint name="left_wheel_joint" type="continuous">
+    <origin xyz="0 1 0" rpy="0 0 0" />
+    <parent link="base_link" />
+    <child link="left_wheel_link" />
+    <axis xyz="0 1 0" rpy="0 0 0" />
+    <limit effort="100" velocity="1.0"/>
+  </joint>
+  <joint name="right_wheel_joint" type="continuous">
+    <origin xyz="0 -1 0" rpy="0 0 0" />
+    <parent link="base_link" />
+    <child link="right_wheel_link" />
+    <axis xyz="0 1 0" rpy="0 0 0" />
+    <limit effort="100" velocity="1.0"/>
+  </joint>
+  <link name="left_wheel_link" />
+  <link name="right_wheel_link" />
   <joint name="ankle_joint" type="revolute">
     <origin xyz="0 0 0.136726" rpy="0 0 0" />
@@ -88,3 +104,4 @@
     </visual>
   </link>
+  <xacro:include filename="$(find r2_control)/urdf/r2.control.urdf.xacro" />
 </robot>

Commit message: Added linear actuator for the center leg.  Updated static script to use it

File: r2_description/urdf/r2.urdf.xacro (robot description, xacro)
@@ -74,8 +74,10 @@
     </visual>
   </link>
-  <joint name="center_leg_joint" type="fixed">
+  <joint name="center_leg_joint" type="prismatic">
     <origin xyz="0 0 -0.56548" rpy="0 0 0" />
     <parent link="body_link" />
     <child link="center_leg_link" />
+    <axis xyz="0 0 1" rpy="0 0 0" />
+    <limit effort="0" lower="0" upper="0.255" velocity="10.0" />
   </joint>
   <link name="center_leg_link">

Commit message: Added head panels.  Some are articulated

File: r2_description/urdf/r2.urdf.xacro (robot description, xacro)
@@ -67,5 +67,5 @@
   <link name="dome_link">
     <visual>
-      <origin xyz="0 0 -0.829076" rpy="0 0 0" />
+      <origin xyz="0 0 0" rpy="0 0 0" />
       <geometry>
         <mesh filename="package://r2_description/meshes/R2_Dome.stl" scale="0.001 0.001 0.001"/>
@@ -74,4 +74,170 @@
     </visual>
   </link>
+  <!-- HEAD-->
+  <link name="panel_1">
+    <visual>
+      <origin xyz="0 0 0" rpy="0 0 0" />
+      <geometry>
+        <mesh filename="package://r2_description/meshes/Panel1.stl" scale="0.001 0.001 0.001"/>
+      </geometry>
+      <material name="Blu"> <color rgba="0.1 0.1 0.9 1.0"/> </material>
+    </visual>
+  </link>
+  <joint name="panel_1_joint" type="fixed">
+    <origin xyz="0.0 0.0 0.0" rpy="0 0 0" />
+    <parent link="dome_link" />
+    <child link="panel_1" />
+  </joint>
+  <link name="panel_2">
+    <visual>
+      <origin xyz="0 0 0" rpy="0 0 0" />
+      <geometry>
+        <mesh filename="package://r2_description/meshes/Panel2.stl" scale="0.001 0.001 0.001"/>
+      </geometry>
+      <material name="Blu"> <color rgba="0.1 0.1 0.9 1.0"/> </material>
+    </visual>
+  </link>
+  <joint name="panel_2_joint" type="fixed">
+    <origin xyz="0.0 0.0 0.0" rpy="0 0 0" />
+    <parent link="dome_link" />
+    <child link="panel_2" />
+  </joint>
+  <link name="panel_3">
+    <visual>
+      <origin xyz="0 0 0" rpy="0 0 0" />
+      <geometry>
+        <mesh filename="package://r2_description/meshes/Panel3.stl" scale="0.001 0.001 0.001"/>
+      </geometry>
+      <material name="Blu"> <color rgba="0.1 0.1 0.9 1.0"/> </material>
+    </visual>
+  </link>
+  <joint name="panel_3_joint" type="fixed">
+    <origin xyz="0.0 0.0 0.0" rpy="0 0 0" />
+    <parent link="dome_link" />
+    <child link="panel_3" />
+  </joint>
+  <link name="panel_4">
+    <visual>
+      <origin xyz="0 0 0" rpy="0 0 0" />
+      <geometry>
+        <mesh filename="package://r2_description/meshes/Panel4.stl" scale="0.001 0.001 0.001"/>
+      </geometry>
+      <material name="Blu"> <color rgba="0.1 0.1 0.9 1.0"/> </material>
+    </visual>
+  </link>
+  <joint name="panel_4_joint" type="fixed">
+    <origin xyz="0.0 0.0 0.0" rpy="0 0 0" />
+    <parent link="dome_link" />
+    <child link="panel_4" />
+  </joint>
+  <link name="panel_5">
+    <visual>
+      <origin xyz="0 0 0" rpy="0 0 0" />
+      <geometry>
+        <mesh filename="package://r2_description/meshes/Panel5.stl" scale="0.001 0.001 0.001"/>
+      </geometry>
+      <material name="Blu"> <color rgba="0.1 0.1 0.9 1.0"/> </material>
+    </visual>
+  </link>
+  <joint name="panel_5_joint" type="fixed">
+    <origin xyz="0.0 0.0 0.0" rpy="0 0 0" />
+    <parent link="dome_link" />
+    <child link="panel_5" />
+  </joint>
+  <link name="panel_6">
+    <visual>
+      <origin xyz="0 0 0" rpy="0 0 0" />
+      <geometry>
+        <mesh filename="package://r2_description/meshes/Panel6.stl" scale="0.001 0.001 0.001"/>
+      </geometry>
+      <material name="Blu"> <color rgba="0.1 0.1 0.9 1.0"/> </material>
+    </visual>
+  </link>
+  <joint name="panel_6_joint" type="fixed">
+    <origin xyz="0.0 0.0 0.0" rpy="0 0 0" />
+    <parent link="dome_link" />
+    <child link="panel_6" />
+  </joint>
+  <link name="panel_7">
+    <visual>
+      <origin xyz="0 0 0" rpy="0 0 0" />
+      <geometry>
+        <mesh filename="package://r2_description/meshes/PanelTop.stl" scale="0.001 0.001 0.001"/>
+      </geometry>
+      <material name="Blu"> <color rgba="0.1 0.1 0.9 1.0"/> </material>
+    </visual>
+  </link>
+  <joint name="panel_7_joint" type="revolute">
+    <origin xyz="0.000835055 -0.135122 0.203276" rpy="0 0 1.5707" />
+    <parent link="dome_link" />
+    <child link="panel_7" />
+    <axis xyz="0 -1 0" rpy="0 0 0" />
+    <limit effort="0" lower="0" upper="0.7" velocity="10.0" />
+  </joint>
+  <link name="panel_8">
+    <visual>
+      <origin xyz="0 0 0" rpy="0 0 0" />
+      <geometry>
+        <mesh filename="package://r2_description/meshes/PanelTop.stl" scale="0.001 0.001 0.001"/>
+      </geometry>
+      <material name="Blu"> <color rgba="0.1 0.1 0.9 1.0"/> </material>
+    </visual>
+  </link>
+  <joint name="panel_8_joint" type="revolute">
+    <origin xyz="0.116446 -0.0678808 0.203276" rpy="0 0 2.6180" />
+    <parent link="dome_link" />
+    <child link="panel_8" />
+    <axis xyz="0 -1 0" rpy="0 0 0" />
+    <limit effort="0" lower="0" upper="0.7" velocity="10.0" />
+  </joint>
+  <link name="panel_9">
+    <visual>
+      <origin xyz="0 0 0" rpy="0 0 0" />
+      <geometry>
+        <mesh filename="package://r2_description/meshes/PanelTop.stl" scale="0.001 0.001 0.001"/>
+      </geometry>
+      <material name="Blu"> <color rgba="0.1 0.1 0.9 1.0"/> </material>
+    </visual>
+  </link>
+  <joint name="panel_9_joint" type="revolute">
+    <origin xyz="0.116446 0.0678808 0.203276" rpy="0 0 3.6652" />
+    <parent link="dome_link" />
+    <child link="panel_9" />
+    <axis xyz="0 -1 0" rpy="0 0 0" />
+    <limit effort="0" lower="0" upper="0.7" velocity="10.0" />
+  </joint>
+  <link name="panel_10">
+    <visual>
+      <origin xyz="0 0 0" rpy="0 0 0" />
+      <geometry>
+        <mesh filename="package://r2_description/meshes/PanelTop.stl" scale="0.001 0.001 0.001"/>
+      </geometry>
+      <material name="Blu"> <color rgba="0.1 0.1 0.9 1.0"/> </material>
+    </visual>
+  </link>
+  <joint name="panel_10_joint" type="revolute">
+    <origin xyz="0.000835055 0.135122 0.203276" rpy="0 0 4.7124" />
+    <parent link="dome_link" />
+    <child link="panel_10" />
+    <axis xyz="0 -1 0" rpy="0 0 0" />
+    <limit effort="0" lower="0" upper="0.7" velocity="10.0" />
+  </joint>
+  <link name="panel_11">
+    <visual>
+      <origin xyz="0 0 0" rpy="0 0 0" />
+      <geometry>
+        <mesh filename="package://r2_description/meshes/PanelTop.stl" scale="0.001 0.001 0.001"/>
+      </geometry>
+      <material name="Blu"> <color rgba="0.1 0.1 0.9 1.0"/> </material>
+    </visual>
+  </link>
+  <joint name="panel_11_joint" type="revolute">
+    <origin xyz="-0.116446 -0.0678808 0.203276" rpy="0 0 0.5236" />
+    <parent link="dome_link" />
+    <child link="panel_11" />
+    <axis xyz="0 -1 0" rpy="0 0 0" />
+    <limit effort="0" lower="0" upper="0.7" velocity="10.0" />
+  </joint>
+  <!-- /HEAD -->
   <joint name="center_leg_joint" type="prismatic">
     <origin xyz="0 0 -0.56548" rpy="0 0 0" />

Commit message: Added zed wrapper and added zedxmini to urdf

File: r2_description/urdf/r2.urdf.xacro (robot description, xacro)
@@ -1,4 +1,5 @@
 <?xml version="1.0"?>
 <robot name="r2" xmlns:xacro="http://ros.org/wiki/xacro">
+  <xacro:include filename="$(find zed_description)/urdf/zed_macro.urdf.xacro" />
   <link name="base_link">
     <visual>
@@ -58,4 +59,12 @@
     </visual>
   </link>
+  <xacro:zed_camera name="zedxm" model="zedxm" >
+    <origin xyz="0 0 0" rpy="0 0 0"/>
+  </xacro:zed_camera>
+  <joint name="zed_camera_joint" type="fixed">
+    <origin xyz="0.216157 0 -0.298453" rpy="0 0 0" />
+    <parent link="body_link" />
+    <child link="zedxm_camera_link" />
+  </joint>
   <joint name="neck_joint" type="revolute">
     <origin xyz="0 0 0.12687" rpy="0 0 0" />
